File: 4_4Keyboard/_autosave-4_4Keyboard.sch (KiCad schematic (older format))
At the start: 62 parts

Commit message: added code
Parts:
- gave numbers to parts that had none: 2
Changed lines of the file:
@@
 	2950 7650 3350 7650
 $Comp
-L pspice:CAP C?
+L pspice:CAP 10nF
 U 1 1 5D9E1751
 P 3350 7400
-F 0 "C?" H 3528 7446 50  0000 L CNN
+F 0 "10nF" H 3528 7446 50  0000 L CNN
 F 1 "CAP" H 3528 7355 50  0000 L CNN
 F 2 "" H 3350 7400 50  0001 C CNN
@@
 Connection ~ 2950 7150
 $Comp
-L pspice:CAP C?
+L pspice:CAP 1uF
 U 1 1 5D9E234F
 P 2950 7400
-F 0 "C?" H 3128 7446 50  0000 L CNN
+F 0 "1uF" H 3128 7446 50  0000 L CNN
 F 1 "CAP" H 3128 7355 50  0000 L CNN
 F 2 "" H 2950 7400 50  0001 C CNN
