File: 4_4Keyboard/4_4Keyboard.sch (KiCad schematic (older format))
At the start: 55 parts

Commit message: Patrick Commit
Parts:
- removed SW? (x19): SW_Push, symbol Switch:SW_Push
- added 100nF1, 10nF1, 1uF1, 4.7uF1: CAP, Capacitor_SMD:C_0603_1608Metric, symbol pspice:CAP
- added C3, C4, C5, C6: 0.1 uF, Capacitor_SMD:C_0603_1608Metric, symbol Device:C
- added FB1: Ferrite_Bead 600, Inductor_SMD:L_0603_1608Metric, symbol Device:Ferrite_Bead
- added KEY_SWITCH10, KEY_SWITCH11, KEY_SWITCH12, KEY_SWITCH13, KEY_SWITCH14, KEY_SWITCH15, KEY_SWITCH16, KEY_SWITCH17, KEY_SWITCH18, KEY_SWITCH19, KEY_SWITCH2, KEY_SWITCH20, KEY_SWITCH3, KEY_SWITCH4, KEY_SWITCH5, KEY_SWITCH6, KEY_SWITCH7, KEY_SWITCH8, KEY_SWITCH9: SW_Push, Button_Switch_Keyboard:SW_Cherry_MX_1.00u_PCB, symbol Switch:SW_Push
- C1, C2: renamed from C?; footprint (none) -> Capacitor_SMD:C_0603_1608Metric
- D1, D2, D3, D4: renamed from D?; footprint (none) -> LED_THT:LED_D5.0mm
- J1: renamed from J?; footprint (none) -> Connector_USB:USB_Mini-B_Lumberg_2486_01_Horizontal
- J2: renamed from J?; footprint (none) -> Connector_PinHeader_2.54mm:PinHeader_1x06_P2.54mm_Vertical
- J3: renamed from J?; footprint (none) -> Connector_PinHeader_2.54mm:PinHeader_2x07_P2.54mm_Vertical
- KEY_SWITCH1: renamed from SW?; footprint (none) -> Button_Switch_Keyboard:SW_Cherry_MX_1.00u_PCB
- R1, R2: renamed from R?; footprint (none) -> Resistor_THT:R_Axial_DIN0207_L6.3mm_D2.5mm_P7.62mm_Horizontal
- SW1: renamed from SW?; value SW_Push -> DOOM KEY; footprint (none) -> Button_Switch_Keyboard:SW_Cherry_MX_1.00u_PCB
- gave numbers to parts that had none: 23
Connections:
- net GND: now also C1.1, 100nF1.2, 10nF1.2, 1uF1.2, 4.7uF1.2, C3.1, C4.1, C6.2; no longer C1.2
- net ROW_0: now also KEY_SWITCH11.1, KEY_SWITCH16.1, KEY_SWITCH6.1
- net ROW_1: now also KEY_SWITCH12.1, KEY_SWITCH17.1, KEY_SWITCH2.1, KEY_SWITCH7.1
- net ROW_2: now also KEY_SWITCH13.1, KEY_SWITCH18.1, KEY_SWITCH3.1, KEY_SWITCH8.1
- net ROW_3: now also KEY_SWITCH14.1, KEY_SWITCH19.1, KEY_SWITCH4.1, KEY_SWITCH9.1
- net ROW_4: now also KEY_SWITCH10.1, KEY_SWITCH15.1, KEY_SWITCH20.1, KEY_SWITCH5.1
- net VCC_3_3: now also U1.1 (VBAT), U1.32 (VDD), U1.48 (VDDUSB), 100nF1.1, 4.7uF1.1, C3.2, C4.2, C6.1, FB1.1
- net VCC_3_3A: now reaches U1.13 (VDDA)
- net VCC_3_3A: now also U2.2 (VOUT), 10nF1.1, 1uF1.1, FB1.2
- net at U1.64 (VDD): now also C5.2
- net at SW1.2, U1.7 (NRST): now also C1.2; no longer C1.1
- net at D7.2 (A): now also KEY_SWITCH2.2
- net at D8.2 (A): now also KEY_SWITCH3.2
- net at D9.2 (A): now also KEY_SWITCH4.2
- net at D11.2 (A): now also KEY_SWITCH6.2
- net at D12.2 (A): now also KEY_SWITCH7.2
- net at D13.2 (A): now also KEY_SWITCH8.2
- net at D14.2 (A): now also KEY_SWITCH9.2
- net at D16.2 (A): now also KEY_SWITCH11.2
- net at D17.2 (A): now also KEY_SWITCH12.2
- net at D18.2 (A): now also KEY_SWITCH13.2
- net at D19.2 (A): now also KEY_SWITCH14.2
- net at D21.2 (A): now also KEY_SWITCH16.2
- net at D22.2 (A): now also KEY_SWITCH17.2
- net at D23.2 (A): now also KEY_SWITCH18.2
- net at D24.2 (A): now also KEY_SWITCH19.2
- net at D10.2 (A): now also KEY_SWITCH5.2
- net at D15.2 (A): now also KEY_SWITCH10.2
- net at D20.2 (A): now also KEY_SWITCH15.2
- net at D25.2 (A): now also KEY_SWITCH20.2
Other:
- moved on the sheet: C1, C2, D1, D2, D3, D4, D5, J1, R1, R2, SW1, U1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

Commit message: Board layout first push
Parts:
- added D6: LED, LED_THT:LED_D5.0mm, symbol Device:LED
- added LED0_R1: LED0_R, Resistor_THT:R_Axial_DIN0207_L6.3mm_D2.5mm_P7.62mm_Horizontal, symbol Device:R
- added LED1_R1: LED1_R, Resistor_THT:R_Axial_DIN0207_L6.3mm_D2.5mm_P7.62mm_Horizontal, symbol Device:R
- added LED2_R1: LED2_R, Resistor_THT:R_Axial_DIN0207_L6.3mm_D2.5mm_P7.62mm_Horizontal, symbol Device:R
- added LED3_R1: LED3_R, Resistor_THT:R_Axial_DIN0207_L6.3mm_D2.5mm_P7.62mm_Horizontal, symbol Device:R
- added LED4_R1: LED4_R, Resistor_THT:R_Axial_DIN0207_L6.3mm_D2.5mm_P7.62mm_Horizontal, symbol Device:R
- FB1: value Ferrite_Bead 600 -> Ferrite Bead
- J2: value Conn_01x06 -> SERIAL WIRE
- J3: value Conn_02x07_Counter_Clockwise -> Pin Breakout
- KEY_SWITCH1: value SW_Push -> R0_C0
- KEY_SWITCH10: value SW_Push -> R4_C1
- KEY_SWITCH11: value SW_Push -> R0_C2
- KEY_SWITCH12: value SW_Push -> R1_C2
- KEY_SWITCH13: value SW_Push -> R2_C2
- KEY_SWITCH14: value SW_Push -> R3_C2
- KEY_SWITCH15: value SW_Push -> R4_C2
- KEY_SWITCH16: value SW_Push -> R0_C3
- KEY_SWITCH17: value SW_Push -> R1_C3
- KEY_SWITCH18: value SW_Push -> R2_C3
- KEY_SWITCH19: value SW_Push -> R3_C3
- KEY_SWITCH2: value SW_Push -> R1_C0
- KEY_SWITCH20: value SW_Push -> R4_C3
- KEY_SWITCH3: value SW_Push -> R2_C0
- KEY_SWITCH4: value SW_Push -> R3_C0
- KEY_SWITCH5: value SW_Push -> R4_C0
- KEY_SWITCH6: value SW_Push -> R0_C1
- KEY_SWITCH7: value SW_Push -> R1_C1
- KEY_SWITCH8: value SW_Push -> R2_C1
- KEY_SWITCH9: value SW_Push -> R3_C1
- renumbered D6 to R0_C0, D11 to R0_C1, D16 to R0_C2, D21 to R0_C3, D7 to R1_C0, D12 to R1_C1, D17 to R1_C2, D22 to R1_C3, D8 to R2_C0, D13 to R2_C1, D18 to R2_C2, D23 to R2_C3, D9 to R3_C0, D14 to R3_C1, D19 to R3_C2, D24 to R3_C3, D10 to R4_C0, D15 to R4_C1, D20 to R4_C2, D25 to R4_C3, SW1 to RESET1
Connections:
- net D_PIN_10: now also J3.11 (Pin_11); no longer J3.12 (Pin_12)
- net D_PIN_11: now also J3.10 (Pin_10); no longer J3.13 (Pin_13)
- net D_PIN_12: now also J3.9 (Pin_9); no longer J3.14 (Pin_14)
- net D_PIN_7: now also J3.14 (Pin_14); no longer J3.9 (Pin_9)
- net D_PIN_8: now also J3.13 (Pin_13); no longer J3.10 (Pin_10)
- net D_PIN_9: now also J3.12 (Pin_12); no longer J3.11 (Pin_11)
- net FS_DM: now also D5.1; no longer D5.3
- net FS_DP: now also D5.3; no longer D5.1
- net GND: now also C5.1, D6.1 (K)
- net VCC_3_3: now also C5.2, U1.64 (VDD)
- net VCC_3_3A: now also LED0_R1.2
- net at U1.56 (PB4): now also LED1_R1.2; no longer D1.2 (A)
- net at U1.57 (PB5): now also LED2_R1.2; no longer D2.2 (A)
- net at U1.58 (PB6): now also LED3_R1.2; no longer D3.2 (A)
- net at U1.59 (PB7): now also LED4_R1.2; no longer D4.2 (A)
- new net: D1.2 (A), LED1_R1.1
- new net: D2.2 (A), LED2_R1.1
- new net: D3.2 (A), LED3_R1.1
- new net: D4.2 (A), LED4_R1.1
- new net: D6.2 (A), LED0_R1.1
Other:
- moved on the sheet: C5

Commit message: Board Design Start
Parts:
- removed J3: Pin Breakout, Connector_PinHeader_2.54mm:PinHeader_2x07_P2.54mm_Vertical, symbol Connector_Generic:Conn_02x07_Counter_Clockwise
- added J3, J4: Conn_01x07, Connector_PinHeader_2.54mm:PinHeader_1x07_P2.54mm_Vertical, symbol Connector_Generic:Conn_01x07
Connections:
- net D_PIN_1 is gone; now on net D_PIN_9: U1.24 (PC4)
- net D_PIN_2 is gone; now on net D_PIN_11: U1.23 (PA7)
- net D_PIN_10: now also U1.17 (PA3), J4.5 (Pin_5); no longer U1.29 (PB10)
- net D_PIN_11: now also J3.6 (Pin_6); no longer U1.30 (PB11)
- net D_PIN_12: now also U1.20 (PA4), J4.6 (Pin_6); no longer U1.25 (PC5)
- net D_PIN_3: now also U1.27 (PB1), J3.2 (Pin_2); no longer U1.22 (PA6)
- net D_PIN_4: now also U1.28 (PB2), J4.2 (Pin_2); no longer U1.21 (PA5)
- net D_PIN_5: now also U1.26 (PB0), J3.3 (Pin_3); no longer U1.20 (PA4)
- net D_PIN_6: now also U1.29 (PB10), J4.3 (Pin_3); no longer U1.17 (PA3)
- net D_PIN_7: now also U1.25 (PC5), J3.4 (Pin_4); no longer U1.26 (PB0)
- net D_PIN_8: now also U1.30 (PB11), J4.4 (Pin_4); no longer U1.27 (PB1)
- net D_PIN_9: now also J3.5 (Pin_5); no longer U1.28 (PB2)
- net GND: now also J3.1 (Pin_1)
- net VCC_3_3: now also J4.1 (Pin_1)
- new net D_PIN_13: J3.7 (Pin_7), U1.22 (PA6)
- new net D_PIN_14: J4.7 (Pin_7), U1.21 (PA5)
Changed lines of the file:
@@
 $EndComp
 Text Label 3750 2750 0    50   ~ 0
+D_PIN_10
+Text Label 3750 2950 0    50   ~ 0
+D_PIN_14
+Text Label 3750 3050 0    50   ~ 0
+D_PIN_13
+Text Label 3750 3150 0    50   ~ 0
+D_PIN_11
+Text Label 1800 4550 0    50   ~ 0
+D_PIN_9
+Text Label 1800 4650 0    50   ~ 0
+D_PIN_7
+Text Label 3800 4150 0    50   ~ 0
+D_PIN_5
+Text Label 3800 4250 0    50   ~ 0
+D_PIN_3
+Text Label 3650 4350 0    50   ~ 0
+D_PIN_4
+Text Label 3800 5200 0    50   ~ 0
 D_PIN_6
-Text Label 3750 2850 0    50   ~ 0
-D_PIN_5
-Text Label 3750 2950 0    50   ~ 0
-D_PIN_4
-Text Label 3750 3050 0    50   ~ 0
-D_PIN_3
-Text Label 3750 3150 0    50   ~ 0
-D_PIN_2
-Text Label 1800 4550 0    50   ~ 0
-D_PIN_1
-Text Label 1800 4650 0    50   ~ 0
-D_PIN_12
-Text Label 3800 4150 0    50   ~ 0
-D_PIN_7
-Text Label 3800 4250 0    50   ~ 0
+Text Label 3800 5300 0    50   ~ 0
 D_PIN_8
-Text Label 3650 4350 0    50   ~ 0
-D_PIN_9
-Text Label 3800 5200 0    50   ~ 0
-D_PIN_10
-Text Label 3800 5300 0    50   ~ 0
-D_PIN_11
 Wire Wire Line
 	3550 2750 3750 2750
@@
 	3550 4150 3800 4150
 Text Label 9300 1400 0    50   ~ 0
-D_PIN_6
+D_PIN_11
 Wire Wire Line
 	9300 1400 9800 1400
 Text Label 9300 1300 0    50   ~ 0
-D_PIN_5
+D_PIN_9
 Wire Wire Line
 	9300 1300 9800 1300
 Text Label 9300 1200 0    50   ~ 0
-D_PIN_4
+D_PIN_7
 Wire Wire Line
 	9300 1200 9800 1200
 Text Label 9300 1100 0    50   ~ 0
-D_PIN_3
+D_PIN_5
 Wire Wire Line
 	9300 1100 9800 1100
 Text Label 9300 1000 0    50   ~ 0
-D_PIN_2
+D_PIN_3
 Wire Wire Line
 	9300 1000 9800 1000
-Text Label 9300 900  0    50   ~ 0
-D_PIN_1
-Wire Wire Line
-	9300 900  9800 900
 Text Label 10600 1400 0    50   ~ 0
 D_PIN_12
 Text Label 10600 1300 0    50   ~ 0
-D_PIN_11
+D_PIN_10
 Text Label 10600 1200 0    50   ~ 0
-D_PIN_10
+D_PIN_8
 Text Label 10600 1100 0    50   ~ 0
-D_PIN_9
+D_PIN_6
 Text Label 10600 1000 0    50   ~ 0
-D_PIN_8
+D_PIN_4
 Text Label 10600 900  0    50   ~ 0
-D_PIN_7
+VCC_3_3
 Wire Wire Line
 	10300 1400 10600 1400
@@
 Wire Wire Line
 	4300 4750 4300 4850
-$Comp
-L Connector_Generic:Conn_02x07_Counter_Clockwise J3
-U 1 1 5D9F22FF
-P 10000 1200
-F 0 "J3" H 10050 1717 50  0000 C CNN
-F 1 "Pin Breakout" H 10050 1626 50  0000 C CNN
-F 2 "Connector_PinHeader_2.54mm:PinHeader_2x07_P2.54mm_Vertical" H 10000 1200 50  0001 C CNN
-F 3 "~" H 10000 1200 50  0001 C CNN
-	1    10000 1200
-	1    0    0    -1
-$EndComp
 Text Label 9300 1500 0    50   ~ 0
-VCC_3_3
+D_PIN_13
 Wire Wire Line
 	9300 1500 9800 1500
@@
 L power:GND #PWR0105
 U 1 1 5DA6FBDF
-P 10600 1500
-F 0 "#PWR0105" H 10600 1250 50  0001 C CNN
-F 1 "GND" V 10605 1372 50  0000 R CNN
-F 2 "" H 10600 1500 50  0001 C CNN
-F 3 "" H 10600 1500 50  0001 C CNN
-	1    10600 1500
-	0    -1   -1   0
+P 9700 900
+F 0 "#PWR0105" H 9700 650 50  0001 C CNN
+F 1 "GND" V 9705 772 50  0000 R CNN
+F 2 "" H 9700 900 50  0001 C CNN
+F 3 "" H 9700 900 50  0001 C CNN
+	1    9700 900
+	0    1    -1   0
 $EndComp
 Wire Wire Line
@@
 Wire Wire Line
 	2950 1300 2950 2250
+$Comp
+L Connector_Generic:Conn_01x07 J3
+U 1 1 5D7F47A8
+P 10000 1200
+F 0 "J3" H 10080 1242 50  0000 L CNN
+F 1 "Conn_01x07" H 10080 1151 50  0000 L CNN
+F 2 "Connector_PinHeader_2.54mm:PinHeader_1x07_P2.54mm_Vertical" H 10000 1200 50  0001 C CNN
+F 3 "~" H 10000 1200 50  0001 C CNN
+	1    10000 1200
+	1    0    0    -1
+$EndComp
+$Comp
+L Connector_Generic:Conn_01x07 J4
+U 1 1 5D7F67F5
+P 10100 1200
+F 0 "J4" H 10018 1717 50  0000 C CNN
+F 1 "Conn_01x07" H 10018 1626 50  0000 C CNN
+F 2 "Connector_PinHeader_2.54mm:PinHeader_1x07_P2.54mm_Vertical" H 10100 1200 50  0001 C CNN
+F 3 "~" H 10100 1200 50  0001 C CNN
+	1    10100 1200
+	-1   0    0    -1
+$EndComp
+Wire Wire Line
+	9700 900  9800 900
+Text Label 3750 2850 0    50   ~ 0
+D_PIN_12
+Text Label 10600 1500 0    50   ~ 0
+D_PIN_14
 $EndSCHEMATC
